File: ISO-macro.sch (KiCad schematic (older format))
At the start: 20 parts, among them J1 USB_C_Receptacle_USB2.0, SW1 SW_SPST, SW2 SW_SPST, SW3 SW_SPST, SW4 SW_SPST, SW5 SW_SPST, SW6 SW_SPST, SW7 SW_SPST, SW8 Rotary_Encoder_Switch, SW9 SW_SPST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

Commit message: add backlights, connect things
Parts:
- added C2, C3: 100n, Capacitor_SMD:C_0402_1005Metric, symbol Device:C
- added C4, C5, C6: 100nF, Capacitor_SMD:C_0402_1005Metric, symbol Device:C
- added D1, D2, D3: WS2812B, LED_SMD:LED_WS2812B_PLCC4_5.0x5.0mm_P3.2mm, symbol LED:WS2812B
- added R7, R8: 10k, Resistor_SMD:R_0402_1005Metric, symbol Device:R
- SW8: value Rotary_Encoder_Switch -> EC11
Connections:
- net GND: now also SW8.C, C2.2, C3.2, C4.2, C5.2, C6.2, D1.3 (VSS), D2.3 (VSS), D3.3 (VSS)
- net VCC: now also C4.1, C5.1, C6.1, D1.1 (VDD), D2.1 (VDD), D3.1 (VDD), R7.1, R8.1
- net EncA: now reaches SW8.A
- net EncA: now also C3.1, R8.2
- net EncB: now reaches SW8.B
- net EncB: now also C2.1, R7.2
- new net: D1.2 (DOUT), D2.4 (DIN)
- new net: D2.2 (DOUT), D3.4 (DIN)
- new net LED: D1.4 (DIN)
- no-connect marks 0 -> 3
