File: ISO-macro.kicad_pcb (KiCad board)
At the start: 2 copper layers, 105.9 x 38.1 mm, 26 parts, among them J1 USB_C_Receptacle_USB2.0, SW1 SW_SPST, SW2 SW_SPST, SW3 SW_SPST, SW4 SW_SPST, SW5 SW_SPST, SW6 SW_SPST, SW7 SW_SPST, SW8 EC11, SW9 SW_SPST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

Commit message: wip
Parts:
- moved SW9 70.0 mm to (118.7, 89.3), turned to 180 degrees
- moved R1 12.5 mm to (119.4, 85.7), turned to 270 degrees
- moved R4 5.79 mm to (125.9, 93.6), turned to 180 degrees
- moved C4 2.87 mm to (139.1, 78.3)
- moved R6 2.17 mm to (124.2, 67.7)
- moved C1 1.87 mm to (124.5, 83.9), turned to 90 degrees
- moved Y1 1.75 mm to (131.2, 87.1), turned to 270 degrees
- moved R2 1.14 mm to (122.6, 71.8)
- moved R3 1.14 mm to (123.7, 71.8)
- moved R5 1.14 mm to (117.5, 68.6)
- moved C5 0.38 mm to (173.0, 77.6)
- turned D1 to 270 degrees
- turned D2 to 270 degrees
- turned D3 to 90 degrees
- turned U1 to 180 degrees
Connections:
- D3 pad 2: (no net) -> Net-(D3-Pad2)
- J1 pad A8: (no net) -> Net-(J1-PadA8)
- J1 pad B8: (no net) -> Net-(J1-PadB8)
- SW1 pad 1: GND -> Net-(SW1-Pad1)
- SW2 pad 1: GND -> Net-(SW2-Pad1)
- SW3 pad 1: GND -> Net-(SW3-Pad1)
- SW4 pad 1: GND -> Net-(SW4-Pad1)
- SW5 pad 1: GND -> Net-(SW5-Pad1)
- SW6 pad 1: GND -> Net-(SW6-Pad1)
- SW7 pad 1: GND -> Net-(SW7-Pad1)
- U1 pad 10: (no net) -> Net-(U1-Pad10)
- U1 pad 11: (no net) -> Net-(U1-Pad11)
- U1 pad 12: (no net) -> Net-(U1-Pad12)
- U1 pad 14: Net-(SW7-Pad2) -> Net-(U1-Pad14)
- U1 pad 15: Net-(SW6-Pad2) -> Net-(U1-Pad15)
- U1 pad 17: (no net) -> Net-(U1-Pad17)
- U1 pad 18: (no net) -> Net-(U1-Pad18)
- U1 pad 19: Net-(SW2-Pad2) -> Net-(U1-Pad19)
- U1 pad 20: /encsw -> Net-(U1-Pad20)
- U1 pad 21: (no net) -> Net-(U1-Pad21)
- U1 pad 22: (no net) -> Net-(U1-Pad22)
- U1 pad 23: Net-(SW1-Pad2) -> /encsw
- U1 pad 25: (no net) -> Net-(U1-Pad25)
- U1 pad 26: /EncB -> Net-(U1-Pad26)
- U1 pad 6: Net-(SW3-Pad2) -> /EncB
- U1 pad 7: Net-(SW5-Pad2) -> Net-(U1-Pad7)
- U1 pad 8: (no net) -> Net-(U1-Pad8)
- U1 pad 9: (no net) -> Net-(U1-Pad9)
Routing:
- net VCC: track 0.00 -> 66.9 mm, vias 4 -> 3
- net GND: track 0.00 -> 26.2 mm, vias 5 -> 6
- net /EncB: track 0.00 -> 23.9 mm
- net /EncA: track 0.00 -> 18.0 mm
- net /encsw: track 0.00 -> 16.3 mm
- net Net-(R2-Pad1): track 0.00 -> 15.2 mm
- net Net-(R3-Pad1): track 0.00 -> 15.0 mm
- net /Data-: track 0.00 -> 14.9 mm, vias 0 -> 2
- net Net-(F1-Pad2): track 0.00 -> 10.6 mm
- net /Reset: track 0.00 -> 10.5 mm
- net /Data+: track 0.00 -> 9.50 mm
- net /Res1: track 0.00 -> 3.64 mm
- net /Res2: track 0.00 -> 3.60 mm
- net Net-(J1-PadB5): track 0.00 -> 3.34 mm
- net Net-(J1-PadA5): track 0.00 -> 2.58 mm
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